File: pcb/interface.kicad_sch (KiCad schematic)
At the start: 10 parts, among them J1 AVR-UPDI-6, J2 QWICC, J3 Power In, J4 Power Out

Commit message: Updated frame template
Other:
- company: CRG Makes -> (none)
Changed lines of the file:
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@@
 	(title_block
 		(title "Relay Module")
-		(date "2025-03-22")
-		(rev "1.1")
-		(company "CRG Makes")
-		(comment 1 "Aquarius")
 	)
 	(rectangle
