File: pcb/mcu.kicad_sch (KiCad schematic)
At the start: 19 parts, among them J1 AVR-UPDI-UART-6, U1 ATtiny1616-MNR

Commit message: Changed opto to be a little smaller
Updated to v10
Parts:
- JP2, JP3, JP7, JP8, TP10, TP11, TP12, TP13, TP14, TP3, TP6, TP7, TP8, TP9: value ~ -> (none)
