File: pcb/requirements.kicad_sch (KiCad schematic)
At the start: 15 parts

Commit message: Changed opto to be a little smaller
Updated to v10
Parts:
- LOGO1, LOGO2, LOGO3, LOGO4, LOGO5, LOGO6, LOGO7, S1, S2, S3, S4: value ~ -> (none)
