File: pcb/relay.kicad_sch (KiCad schematic)
At the start: 17 parts, among them K1 PR24-5V-900-1A, P1 MountingHole_Pad, P2 MountingHole_Pad, P3 MountingHole_Pad, P4 MountingHole_Pad, Q1 MMBT3904, U3 LTV-356T

Commit message: Changed opto to be a little smaller
Updated to v10
Parts:
- removed U3: LTV-356T, CRG Makes:SO-4_4.4x3.6mm_P2.54mm, symbol CRG Makes:LTV-356T
- added U3: TLP291, Package_SO:SOIC-4_4.55x2.6mm_P1.27mm, symbol Isolator:TLP291
- JP6, TP1, TP2: value ~ -> (none)
Connections:
- net +3.3V: now also U3.4
- net GND: now also U3.2
- net at R1.2: now also U3.1
- net at R2.1: now also U3.3
